Commit message: feat: add curobo ik solver

File: assets/franka_panda/franka_panda_umi-isaacsim.urdf (robot description, URDF)
Before this commit: robot panda, 12 links, 11 joints
Links:
- added link umi_tcp
Joints:
- added joint umi_tcp_joint: type fixed, parent panda_link7, child umi_tcp, origin xyz=0 0.086 0.327 rpy=0 0 0
